File: test/max7219_high_voltage.sch (EAGLE design)
At the start: 65 parts, among them IC3 UDN2981A, IC4 MAX7219CNG, IC5 ULN2803, IC6 ULN2803, IC7 UDN2981A, IC8 MAX7219CNG

Commit message: Test Sketch für MAX7219 + Transistoren added
Parts:
- removed C4: 10nF, resistor:C-EU025-025X050
- removed D1, D10, D11, D12, D13, D14, D15, D16, D2, D3, D4, D5, D7, D8, D9: (no value), special:7SEG-MCK
- removed IC1, IC2: (no value), uln-udn:ULN2803A
- removed IC3, IC7: UDN2981A, uln-udn:UDN2981A
- removed IC5, IC6: ULN2803, uln-udn:ULN2803A
- removed IC8: MAX7219CNG, maxim:MAX7219CNG
- removed J_BT_BOARD_1: BLUETOOTH_BOARD, Bluetooth HC-05:BLUETOOTH_BOARD
- removed R12, R13, R14, R15, R16, R17, R18, R28, R29, R30, R31, R32, R33, R34, R35, R37: 2k2, resistor:R-EU_0204/7
- removed R20, R21, R22, R23, R24, R25, R26, R27, R3, R4, R5, R6, R7, R8, R9: 22R, resistor:R-EU_0204/7
- removed R36: 10k, resistor:R-EU_0204/7
- removed R38: 1k, resistor:R-EU_0204/7
- added NPN, NPN1: 2N3904, transistor-npn:2N3904
- added PNP: 2N3906, transistor-pnp:2N3906
- added R1: 10k, resistor:R-EU_0204/7
Connections:
- removed net N$1: IC1.O1, IC2.I1, R11.1
- removed net N$10: D3.CK1, D3.CK2, IC2.O2
- removed net N$100: IC4.DOUT, IC8.DIN
- removed net N$104: J_BT_BOARD_1.TX, MODUL1.D0/RX
- removed net N$105: J_BT_BOARD_1.RX, R37.2, R38.2
- removed net N$11: D2.CK1, D2.CK2, IC2.O3
- removed net N$12: D1.CK1, D1.CK2, IC2.O4
- removed net N$14: IC3.O2, R3.1
- removed net N$15: IC3.O3, R4.1
- removed net N$16: D5.CK1, D5.CK2, IC2.O5
- removed net N$18: D7.CK1, D7.CK2, IC2.O7
- removed net N$19: D8.CK1, D8.CK2, IC2.O8
- removed net N$20: IC3.O4, R5.1
- removed net N$21: IC3.O5, R6.1
- removed net N$23: IC3.O6, R7.1
- removed net N$24: IC3.O7, R8.1
- removed net N$25: IC3.O8, R9.1
- removed net N$26: D1.B, D2.B, D3.B, D4.B, D5.B, D6.B, D7.B, D8.B, R3.2
- removed net N$27: D1.C, D2.C, D3.C, D4.C, D5.C, D6.C, D7.C, D8.C, R4.2
- removed net N$28: D1.D, D2.D, D3.D, D4.D, D5.D, D6.D, D7.D, D8.D, R5.2
- removed net N$29: D1.E, D2.E, D3.E, D4.E, D5.E, D6.E, D7.E, D8.E, R6.2
- removed net N$30: D1.DP, D2.DP, D4.DP, D5.DP, D6.DP, D7.DP, D8.DP, R7.2
- removed net N$31: IC1.I1, IC4.DIG0
- removed net N$32: D1.F, D2.F, D3.F, D4.F, D5.F, D6.F, D7.F, D8.F, R9.2
- removed net N$33: D1.G, D2.G, D3.G, D4.G, D5.G, D6.G, D7.G, D8.G, R8.2
- removed net N$34: IC1.I2, IC4.DIG1
- removed net N$35: IC1.I3, IC4.DIG2
- removed net N$36: IC1.I4, IC4.DIG3
- removed net N$37: IC1.I5, IC4.DIG4
- removed net N$38: IC1.I6, IC4.DIG5
- removed net N$39: IC1.I7, IC4.DIG6
- removed net N$4: IC1.O4, IC2.I4, R14.1
- removed net N$40: IC1.I8, IC4.DIG7
- removed net N$42: IC3.I2, IC4.SEGB
- removed net N$43: IC3.I3, IC4.SEGC
- removed net N$44: IC3.I4, IC4.SEGD
- removed net N$45: IC3.I5, IC4.SEGE
- removed net N$46: IC3.I6, IC4.SEGDP
- removed net N$47: IC3.I7, IC4.SEGG
- removed net N$48: IC3.I8, IC4.SEGF
- removed net N$49: MODUL1.D1/TX, R38.1
- removed net N$5: IC1.O5, IC2.I5, R15.1
- removed net N$51: IC5.O1, IC6.I1, R28.1
- removed net N$52: IC5.O2, IC6.I2, R29.1
- removed net N$53: IC5.O3, IC6.I3, R30.1
- removed net N$54: IC5.O4, IC6.I4, R31.1
- removed net N$55: IC5.O5, IC6.I5, R32.1
- removed net N$56: IC5.O6, IC6.I6, R33.1
- removed net N$57: IC5.O7, IC6.I7, R34.1
- removed net N$58: IC5.O8, IC6.I8, R35.1
- removed net N$59: D12.CK1, D12.CK2, IC6.O1
- removed net N$6: IC1.O6, IC2.I6, R16.1
- removed net N$60: D11.CK1, D11.CK2, IC6.O2
- removed net N$61: D10.CK1, D10.CK2, IC6.O3
- removed net N$62: D9.CK1, D9.CK2, IC6.O4
- removed net N$63: D13.CK1, D13.CK2, IC6.O5
- removed net N$64: D14.CK1, D14.CK2, IC6.O6
- removed net N$65: D15.CK1, D15.CK2, IC6.O7
- removed net N$66: D16.CK1, D16.CK2, IC6.O8
- removed net N$67: D10.A, D11.A, D12.A, D13.A, D14.A, D15.A, D16.A, D9.A, R20.2
- removed net N$68: IC7.O1, R20.1
- removed net N$69: IC7.O2, R21.1
- removed net N$7: IC1.O7, IC2.I7, R17.1
- removed net N$70: IC7.O3, R22.1
- removed net N$71: IC7.O4, R23.1
- removed net N$72: IC7.O5, R24.1
- removed net N$73: IC7.O6, R25.1
- removed net N$74: IC7.O7, R26.1
- removed net N$75: IC7.O8, R27.1
- removed net N$76: D10.B, D11.B, D12.B, D13.B, D14.B, D15.B, D16.B, D9.B, R21.2
- removed net N$77: D10.C, D11.C, D12.C, D13.C, D14.C, D15.C, D16.C, D9.C, R22.2
- removed net N$78: D10.D, D11.D, D12.D, D13.D, D14.D, D15.D, D16.D, D9.D, R23.2
- removed net N$79: D10.E, D11.E, D12.E, D13.E, D14.E, D15.E, D16.E, D9.E, R24.2
- removed net N$8: IC1.O8, IC2.I8, R18.1
- removed net N$80: D10.F, D11.F, D12.F, D13.F, D14.F, D15.F, D16.F, D9.F, R27.2
- removed net N$81: D10.G, D11.G, D12.G, D13.G, D14.G, D15.G, D16.G, D9.G, R26.2
- removed net N$82: D10.DP, D12.DP, D13.DP, D14.DP, D15.DP, D16.DP, D9.DP, R25.2
- removed net N$83: IC5.I1, IC8.DIG0
- removed net N$84: IC5.I2, IC8.DIG1
- removed net N$85: IC5.I3, IC8.DIG2
- removed net N$86: IC5.I4, IC8.DIG3
- removed net N$87: IC5.I5, IC8.DIG4
- removed net N$88: IC5.I6, IC8.DIG5
- removed net N$89: IC5.I7, IC8.DIG6
- removed net N$9: D4.CK1, D4.CK2, IC2.O1
- removed net N$90: IC5.I8, IC8.DIG7
- removed net N$91: IC7.I1, IC8.SEGA
- removed net N$92: IC7.I2, IC8.SEGB
- removed net N$93: IC7.I3, IC8.SEGC
- removed net N$94: IC7.I4, IC8.SEGD
- removed net N$95: IC7.I5, IC8.SEGE
- removed net N$96: IC7.I6, IC8.SEGDP
- removed net N$97: IC7.I7, IC8.SEGG
- removed net N$98: IC7.I8, IC8.SEGF
- removed net N$99: IC8.ISET, R36.2
- net 3.3V: now also NPN.C, NPN1.C, R1.1; no longer C4.2, IC1.GND, IC2.GND, IC3.GND, IC5.GND, IC6.GND, IC7.GND, IC8.GND@1, IC8.GND@2, J_BT_BOARD_1.GND, R37.1
- net N$101: no longer IC8.CLK
- net N$102: no longer IC8.LOAD
- net N$13: now also PNP.C, R1.2; no longer IC3.O1
- net N$17: now also NPN1.E; no longer IC2.O6
- net N$2: now also IC4.DIG0, NPN.B; no longer IC1.O2, IC2.I2, R12.1
- net N$22: no longer D1.A, D2.A, D3.A, D4.A, D5.A, D7.A, D8.A
- net N$3: now also NPN.E, NPN1.B, R11.1; no longer IC1.O3, IC2.I3, R13.1
- net N$41: now also PNP.B; no longer IC3.I1
- net VCC: now also PNP.E; no longer C4.1, IC3.VS, IC8.VCC, J_BT_BOARD_1.VCC, R12.2, R13.2, R14.2, R15.2, R16.2, R17.2, R18.2, R28.2, R29.2, R30.2, R31.2, R32.2, R33.2, R34.2, R35.2, R36.1
Other:
- moved on the sheet: C3, D6, IC4, R11, R19, R2
