File: ideas/No1/#1_routed.sch (EAGLE design)
At the start: 17 parts, among them IC1 ULN2803, IC2 ULN2803, IC3 TD620831A, IC4 TD620831A, U1 SN74HC595N, U2 SN74HC595N, U3 SN74HC595N, U4 SN74HC595N

Commit message: 1_route_1register.sch
Parts:
- added D1: 1N4004, diode:1N4004
- added U$2: DC-DC-STEP-DOWN-LM2596, diy-modules_lm2596:DC-DC-STEP-DOWN-LM2596
Connections:
- removed net N$73: IC4.I2, U3.QB
- removed net N$74: IC4.I3, U3.QC
- removed net N$75: IC4.I4, U3.QD
- removed net N$76: IC4.I5, U3.QE
- removed net N$78: IC4.I7, U3.QG
- removed net N$83: IC1.I1, U4.QA
- removed net N$84: IC1.I2, U4.QB
- removed net N$85: IC1.I3, U4.QC
- removed net N$86: IC1.I4, U4.QD
- removed net N$87: IC1.I5, U4.QE
- removed net N$88: IC1.I6, U4.QF
- removed net N$89: IC1.I7, U4.QG
- removed net N$90: IC1.I8, U4.QH
- new net 24V: IC3.VS, IC4.VS, U$2.IN+
- new net GND: C1.1, C2.-, C3.1, C4.1, C5.1, C6.2, IC1.GND, IC2.GND, IC3.GND, IC4.GND, U$1.GND, U1.GND, U2.GND, U3.GND, U4.GND
- new net N$25: IC4.I1, U1.QH
- new net N$27: IC4.I2, U1.QG
- new net N$29: IC4.I3, U1.QF
- new net N$32: IC4.I5, U1.QD
- new net N$55: IC3.I7, U3.QB
- new net N$56: IC3.I8, U3.QA
- new net N$58: IC1.I2, U4.QG
- new net N$60: IC1.I3, U4.QF
- new net N$62: IC1.I4, U4.QE
- new net N$64: IC1.I5, U4.QD
- new net N$65: IC1.I6, U4.QC
- new net N$66: IC1.I7, U4.QB
- new net N$67: IC1.I8, U4.QA
- new net N$69: D1.A, U$2.OUT+
- net 3.3V: now also U$2.IN-, U$2.OUT-; no longer C1.1, C2.-, C3.1, C4.1, C5.1, C6.2, IC1.GND, IC2.GND, IC3.GND, IC4.GND, U$1.GND, U1.GND, U2.GND, U3.GND, U4.GND
- net N$1: now also U2.QH; no longer U2.QA
- net N$10: now also IC4.O2; no longer IC3.O2
- net N$11: now also IC4.O3; no longer IC3.O3
- net N$12: now also IC4.O4; no longer IC3.O4
- net N$13: now also IC4.O5; no longer IC3.O5
- net N$14: now also IC4.O6; no longer IC3.O6
- net N$15: now also IC4.O7; no longer IC3.O7
- net N$16: now also IC4.O8; no longer IC3.O8
- net N$2: now also U2.QG; no longer U2.QB
- net N$26: now also IC3.O2; no longer IC4.O2
- net N$28: now also IC3.O4; no longer IC4.O4
- net N$3: now also U2.QF; no longer U2.QC
- net N$30: now also IC3.O6; no longer IC4.O6
- net N$31: now also IC4.I4, U1.QE; no longer IC3.I8, U1.QH
- net N$33: now also IC3.O8; no longer IC4.O8
- net N$35: now also IC1.I1, U4.QH; no longer IC4.I8, U3.QH
- net N$4: now also U2.QE; no longer U2.QD
- net N$41: now also IC4.I6, U1.QC; no longer IC3.I1, U1.QA
- net N$42: now also IC4.I7; no longer IC3.I2
- net N$43: now also IC4.I8, U1.QA; no longer IC3.I3, U1.QC
- net N$44: now also IC3.I2, U3.QG; no longer IC3.I4, U1.QD
- net N$45: now also IC3.I3, U3.QF; no longer IC3.I5, U1.QE
- net N$46: now also IC3.I4, U3.QE; no longer IC4.I6, U3.QF
- net N$47: now also IC3.I5, U3.QD; no longer IC3.I7, U1.QG
- net N$48: now also U3.QC; no longer U1.QF
- net N$5: now also U2.QD; no longer U2.QE
- net N$57: now also IC3.O1; no longer IC4.O1
- net N$59: now also IC3.O3; no longer IC4.O3
- net N$6: now also U2.QC; no longer U2.QF
- net N$61: now also IC3.O5; no longer IC4.O5
- net N$63: now also IC3.O7; no longer IC4.O7
- net N$7: now also U2.QB; no longer U2.QG
- net N$72: now also IC3.I1, U3.QH; no longer IC4.I1, U3.QA
- net N$8: now also U2.QA; no longer U2.QH
- net N$9: now also IC4.O1; no longer IC3.O1
- net VCC: now also D1.C; no longer IC3.VS, IC4.VS
Other:
- moved on the sheet: C2, C6, IC3, IC4
